File: board/TinyTrackuino.sch (EAGLE design)
At the start: 16 parts, among them M2 HX1, Q1 PMV20XN, PMV16UN, etc, U1 LM60 int, X1 BU-SMA-V, X2 Vin, X3 LM60 ext, X4 Buzzer

Commit message: Fixing temp sensor silkscreen and gps connector
Connections:
- net 5V: now also GPSCONN.5; no longer GPSCONN.2
- net GND: now also GPSCONN.6; no longer GPSCONN.1
- net GPSPWRCTRL: now also GPSCONN.1; no longer GPSCONN.6
- net GPSVBAT: now also GPSCONN.2; no longer GPSCONN.5
Changed lines of the file:
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@@
 <instance part="S1" gate="1" x="35.56" y="76.2" rot="R270"/>
 <instance part="GND3" gate="1" x="2.54" y="38.1"/>
-<instance part="GND4" gate="1" x="96.52" y="78.74"/>
-<instance part="SUPPLY5" gate="G$1" x="96.52" y="83.82" rot="R270"/>
+<instance part="GND4" gate="1" x="104.14" y="91.44"/>
+<instance part="SUPPLY5" gate="G$1" x="93.98" y="96.52"/>
 </instances>
 <busses>
@@
 </segment>
 <segment>
-<pinref part="GPSCONN" gate="G$1" pin="1"/>
-<wire x1="86.36" y1="81.28" x2="96.52" y2="81.28" width="0.1524" layer="91"/>
-<pinref part="GND4" gate="1" pin="GND"/>
-</segment>
-<segment>
 <pinref part="GND3" gate="1" pin="GND"/>
 <pinref part="U$2" gate="G$1" pin="GND1"/>
@@
 <pinref part="S1" gate="1" pin="S"/>
 </segment>
+<segment>
+<pinref part="GPSCONN" gate="G$1" pin="6"/>
+<pinref part="GND4" gate="1" pin="GND"/>
+<wire x1="86.36" y1="93.98" x2="104.14" y2="93.98" width="0.1524" layer="91"/>
+</segment>
 </net>
 <net name="VIN" class="3">
@@
 </segment>
 <segment>
-<pinref part="GPSCONN" gate="G$1" pin="2"/>
-<wire x1="86.36" y1="83.82" x2="96.52" y2="83.82" width="0.1524" layer="91"/>
-<pinref part="SUPPLY5" gate="G$1" pin="5V"/>
-</segment>
-<segment>
 <pinref part="C1" gate="G$1" pin="+"/>
 <pinref part="SUPPLY1" gate="G$1" pin="5V"/>
@@
 <wire x1="91.44" y1="142.24" x2="96.52" y2="142.24" width="0.1524" layer="91"/>
 </segment>
+<segment>
+<pinref part="GPSCONN" gate="G$1" pin="5"/>
+<wire x1="86.36" y1="91.44" x2="93.98" y2="91.44" width="0.1524" layer="91"/>
+<pinref part="SUPPLY5" gate="G$1" pin="5V"/>
+<wire x1="93.98" y1="91.44" x2="93.98" y2="96.52" width="0.1524" layer="91"/>
+</segment>
 </net>
 <net name="GPSVBAT" class="0">
-<segment>
-<pinref part="GPSCONN" gate="G$1" pin="5"/>
-<wire x1="86.36" y1="91.44" x2="91.44" y2="91.44" width="0.1524" layer="91"/>
-<label x="91.44" y="91.44" size="1.778" layer="95"/>
-</segment>
 <segment>
 <wire x1="121.92" y1="91.44" x2="121.92" y2="99.06" width="0.1524" layer="91"/>
@@
 <pinref part="JP1" gate="G$1" pin="2"/>
 </segment>
+<segment>
+<pinref part="GPSCONN" gate="G$1" pin="2"/>
+<wire x1="86.36" y1="83.82" x2="91.44" y2="83.82" width="0.1524" layer="91"/>
+<label x="91.44" y="83.82" size="1.778" layer="95"/>
+</segment>
 </net>
 <net name="GPSPWRCTRL" class="0">
-<segment>
-<pinref part="GPSCONN" gate="G$1" pin="6"/>
-<wire x1="86.36" y1="93.98" x2="91.44" y2="93.98" width="0.1524" layer="91"/>
-<label x="91.44" y="93.98" size="1.778" layer="95"/>
-</segment>
 <segment>
 <pinref part="U$2" gate="G$1" pin="2"/>
@@
 <label x="5.08" y="35.56" size="1.778" layer="95"/>
 </segment>
-</net>
+<segment>
+<pinref part="GPSCONN" gate="G$1" pin="1"/>
+<wire x1="86.36" y1="81.28" x2="91.44" y2="81.28" width="0.1524" layer="91"/>
+<label x="91.44" y="81.28" size="1.778" layer="95"/>
+</segment>
+</net>

Commit message: Almost final revision of board
Parts:
- C1, C2: device rcl:CPOL-EUE2.5-5 -> adafruit:C-USC3216
Connections:
- net 5V: now also C1.1; no longer C1.+
- net GND: now also C1.2, C2.2; no longer C1.-, C2.-
- net VIN: now also C2.1; no longer C2.+
Changed lines of the file:
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@@
 <layer number="54" name="bGND_GNDA" color="1" fill="9" visible="no" active="no"/>
 <layer number="56" name="wert" color="7" fill="1" visible="no" active="no"/>
+<layer number="57" name="tCAD" color="7" fill="1" visible="no" active="no"/>
 <layer number="60" name="p_dimension" color="6" fill="0" visible="no" active="no"/>
 <layer number="61" name="pt_docu" color="7" fill="0" visible="no" active="no"/>
@@
 <layer number="108" name="tplace-old" color="10" fill="1" visible="yes" active="yes"/>
 <layer number="109" name="ref-old" color="11" fill="1" visible="yes" active="yes"/>
+<layer number="110" name="fp0" color="7" fill="1" visible="no" active="yes"/>
+<layer number="111" name="LPC17xx" color="7" fill="1" visible="yes" active="yes"/>
+<layer number="112" name="tSilk" color="7" fill="1" visible="yes" active="yes"/>
 <layer number="116" name="Patch_BOT" color="9" fill="4" visible="yes" active="yes"/>
 <layer number="121" name="_tsilk" color="7" fill="1" visible="yes" active="yes"/>
 <layer number="122" name="_bsilk" color="7" fill="1" visible="yes" active="yes"/>
+<layer number="123" name="tTestmark" color="7" fill="1" visible="no" active="yes"/>
+<layer number="124" name="bTestmark" color="7" fill="1" visible="no" active="yes"/>
 <layer number="125" name="_tNames" color="7" fill="1" visible="no" active="yes"/>
+<layer number="126" name="_bNames" color="7" fill="1" visible="yes" active="yes"/>
+<layer number="127" name="_tValues" color="7" fill="1" visible="yes" active="yes"/>
+<layer number="128" name="_bValues" color="7" fill="1" visible="yes" active="yes"/>
+<layer number="131" name="tAdjust" color="7" fill="1" visible="no" active="yes"/>
+<layer number="132" name="bAdjust" color="7" fill="1" visible="no" active="yes"/>
 <layer number="144" name="Drill_legend" color="7" fill="1" visible="no" active="yes"/>
 <layer number="146" name="p_Milling" color="3" fill="9" visible="yes" active="yes"/>
 <layer number="147" name="COVER" color="14" fill="1" visible="yes" active="yes"/>
+<layer number="150" name="Notes" color="7" fill="1" visible="no" active="yes"/>
 <layer number="151" name="HeatSink" color="7" fill="1" visible="yes" active="yes"/>
+<layer number="152" name="_bDocu" color="7" fill="1" visible="yes" active="yes"/>
+<layer number="153" name="FabDoc1" color="6" fill="1" visible="no" active="no"/>
+<layer number="154" name="FabDoc2" color="2" fill="1" visible="no" active="no"/>
+<layer number="155" name="FabDoc3" color="7" fill="15" visible="no" active="no"/>
 <layer number="190" name="Comments" color="12" fill="1" visible="yes" active="yes"/>
 <layer number="199" name="Contour" color="7" fill="1" visible="yes" active="yes"/>
@@
 <layer number="223" name="223bmp" color="24" fill="1" visible="no" active="no"/>
 <layer number="224" name="224bmp" color="25" fill="1" visible="no" active="no"/>
+<layer number="248" name="Housing" color="7" fill="1" visible="yes" active="yes"/>
+<layer number="249" name="Edge" color="7" fill="1" visible="yes" active="yes"/>
 <layer number="250" name="Descript" color="3" fill="1" visible="no" active="no"/>
 <layer number="251" name="SMDround" color="12" fill="11" visible="no" active="no"/>
@@
 <part name="GND9" library="supply1" deviceset="GND" device=""/>
 <part name="GND10" library="supply1" deviceset="GND" device=""/>
-<part name="C1" library="rcl" deviceset="CPOL-EU" device="E2.5-5" value="10uF"/>
-<part name="C2" library="rcl" deviceset="CPOL-EU" device="E2.5-5" value="10uF"/>
+<part name="C1" library="adafruit" deviceset="C-US" device="C3216" value="10uF"/>
+<part name="C2" library="adafruit" deviceset="C-US" device="C3216" value="10uF"/>
 <part name="GND" library="supply1" deviceset="GND" device=""/>
 <part name="FRAME1" library="frames" deviceset="DINA4_L" device="" value="v1"/>
@@
 <wire x1="12.7" y1="147.32" x2="12.7" y2="144.78" width="0.1524" layer="91"/>
 <pinref part="GND9" gate="1" pin="GND"/>
-<pinref part="C2" gate="G$1" pin="-"/>
+<pinref part="C2" gate="G$1" pin="2"/>
 </segment>
 <segment>
 <wire x1="33.02" y1="147.32" x2="33.02" y2="144.78" width="0.1524" layer="91"/>
 <pinref part="GND10" gate="1" pin="GND"/>
-<pinref part="C1" gate="G$1" pin="-"/>
+<pinref part="C1" gate="G$1" pin="2"/>
 </segment>
 <segment>
@@
 </segment>
 <segment>
-<pinref part="C2" gate="G$1" pin="+"/>
+<pinref part="C2" gate="G$1" pin="1"/>
 <wire x1="12.7" y1="154.94" x2="12.7" y2="157.48" width="0.1524" layer="91"/>
 <label x="12.7" y="157.48" size="1.778" layer="95" rot="R90" xref="yes"/>
@@
 </segment>
 <segment>
-<pinref part="C1" gate="G$1" pin="+"/>
+<pinref part="C1" gate="G$1" pin="1"/>
 <pinref part="SUPPLY1" gate="G$1" pin="5V"/>
 <wire x1="33.02" y1="157.48" x2="33.02" y2="154.94" width="0.1524" layer="91"/>

Commit message: Possibly final commit for revision 1
Parts:
- removed GPSCONN: JST, SparkFun-Connectors:M06EM406
- added X5: SM06B-SRSS-TB, con-jst2:SM06B-SRSS-TB
- C1, C2: device adafruit:C-USC3216 -> SparkFun-Passives:CAP1206
- R1, R2: device resistor:R-EU_R1206 -> SparkFun-Passives:CAP0603-CAP
Connections:
- net 5V: now also X5-5.S; no longer GPSCONN.5
- net GND: now also X5-6.S; no longer GPSCONN.6
- net GPSPWRCTRL: now also X5-1.S; no longer GPSCONN.1
- net GPSRX: now also X5-4.S; no longer GPSCONN.4
- net GPSTX: now also X5-3.S; no longer GPSCONN.3
- net GPSVBAT: now also X5-2.S; no longer GPSCONN.2
- net RFTX: now also U$2.10; no longer U$2.3
Other:
- moved on the sheet: C1, C2, R1, R2
Changed lines of the file:
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@@
 <part name="GND9" library="supply1" deviceset="GND" device=""/>
 <part name="GND10" library="supply1" deviceset="GND" device=""/>
-<part name="C1" library="adafruit" deviceset="C-US" device="C3216" value="10uF"/>
-<part name="C2" library="adafruit" deviceset="C-US" device="C3216" value="10uF"/>
+<part name="C1" library="SparkFun-Passives" deviceset="CAP" device="1206" value="10uF"/>
+<part name="C2" library="SparkFun-Passives" deviceset="CAP" device="1206" value="10uF"/>
 <part name="GND" library="supply1" deviceset="GND" device=""/>
 <part name="FRAME1" library="frames" deviceset="DINA4_L" device="" value="v1"/>
@@
 <part name="GND14" library="supply1" deviceset="GND" device=""/>
 <part name="GND20" library="supply1" deviceset="GND" device=""/>
-<part name="R1" library="resistor" deviceset="R-EU_" device="R1206" value="10K"/>
-<part name="R2" library="resistor" deviceset="R-EU_" device="R1206" value="3.3K"/>
+<part name="R1" library="SparkFun-Passives" deviceset="CAP" device="0603-CAP" value="10K"/>
+<part name="R2" library="SparkFun-Passives" deviceset="CAP" device="0603-CAP" value="3.3K"/>
 <part name="GND21" library="supply1" deviceset="GND" device=""/>
 <part name="Q1" library="transistor-small-signal" deviceset="BSS123" device="" value="PMV20XN, PMV16UN, etc"/>
@@
 <part name="SUPPLY3" library="SparkFun-Aesthetics" deviceset="5V" device=""/>
 <part name="GND1" library="supply1" deviceset="GND" device=""/>
-<part name="GPSCONN" library="SparkFun-Connectors" deviceset="M06" device="EM406" value="JST"/>
 <part name="GND2" library="supply1" deviceset="GND" device=""/>
 <part name="SUPPLY1" library="SparkFun-Aesthetics" deviceset="5V" device=""/>
@@
 <part name="GND4" library="supply1" deviceset="GND" device=""/>
 <part name="SUPPLY5" library="SparkFun-Aesthetics" deviceset="5V" device=""/>
+<part name="X5" library="con-jst2" deviceset="?M06B-SRSS-TB" device="S"/>
 </parts>
 <sheets>
@@
 <instance part="GND14" gate="1" x="231.14" y="40.64"/>
 <instance part="GND20" gate="1" x="124.46" y="142.24"/>
-<instance part="R1" gate="G$1" x="50.8" y="149.86" rot="R90"/>
-<instance part="R2" gate="G$1" x="50.8" y="132.08" rot="R90"/>
+<instance part="R1" gate="G$1" x="50.8" y="149.86" rot="R180"/>
+<instance part="R2" gate="G$1" x="50.8" y="132.08" rot="R180"/>
 <instance part="GND21" gate="1" x="50.8" y="119.38"/>
 <instance part="Q1" gate="G$1" x="231.14" y="50.8" rot="MR0"/>
@@
 <instance part="SUPPLY3" gate="G$1" x="48.26" y="38.1" rot="R270"/>
 <instance part="GND1" gate="1" x="63.5" y="40.64"/>
-<instance part="GPSCONN" gate="G$1" x="81.28" y="86.36"/>
 <instance part="GND2" gate="1" x="121.92" y="81.28"/>
 <instance part="SUPPLY1" gate="G$1" x="33.02" y="157.48"/>
@@
 <instance part="GND4" gate="1" x="104.14" y="91.44"/>
 <instance part="SUPPLY5" gate="G$1" x="93.98" y="96.52"/>
+<instance part="X5" gate="-1" x="83.82" y="81.28" smashed="yes" rot="R180">
+<attribute name="NAME" x="81.28" y="82.042" size="1.524" layer="95" rot="R180"/>
+</instance>
+<instance part="X5" gate="-2" x="83.82" y="83.82" rot="R180"/>
+<instance part="X5" gate="-3" x="83.82" y="86.36" rot="R180"/>
+<instance part="X5" gate="-4" x="83.82" y="88.9" rot="R180"/>
+<instance part="X5" gate="-5" x="83.82" y="91.44" rot="R180"/>
+<instance part="X5" gate="-6" x="83.82" y="93.98" rot="R180"/>
 </instances>
 <busses>
@@
 <net name="GND" class="0">
 <segment>
-<wire x1="12.7" y1="147.32" x2="12.7" y2="144.78" width="0.1524" layer="91"/>
+<wire x1="12.7" y1="149.86" x2="12.7" y2="144.78" width="0.1524" layer="91"/>
 <pinref part="GND9" gate="1" pin="GND"/>
 <pinref part="C2" gate="G$1" pin="2"/>
 </segment>
 <segment>
-<wire x1="33.02" y1="147.32" x2="33.02" y2="144.78" width="0.1524" layer="91"/>
+<wire x1="33.02" y1="149.86" x2="33.02" y2="144.78" width="0.1524" layer="91"/>
 <pinref part="GND10" gate="1" pin="GND"/>
 <pinref part="C1" gate="G$1" pin="2"/>
@@
 </segment>
 <segment>
-<pinref part="GPSCONN" gate="G$1" pin="6"/>
 <pinref part="GND4" gate="1" pin="GND"/>
 <wire x1="86.36" y1="93.98" x2="104.14" y2="93.98" width="0.1524" layer="91"/>
-</segment>
-</net>
-<net name="VIN" class="3">
+<pinref part="X5" gate="-6" pin="S"/>
+</segment>
+</net>
+<net name="VIN" class="0">
 <segment>
 <wire x1="154.94" y1="58.42" x2="160.02" y2="58.42" width="0.1524" layer="91"/>
@@
 </segment>
 <segment>
-<wire x1="50.8" y1="154.94" x2="50.8" y2="160.02" width="0.1524" layer="91"/>
+<wire x1="50.8" y1="152.4" x2="50.8" y2="160.02" width="0.1524" layer="91"/>
 <label x="50.8" y="160.02" size="1.778" layer="95" xref="yes"/>
 <pinref part="R1" gate="G$1" pin="2"/>
@@
 <segment>
 <pinref part="C2" gate="G$1" pin="1"/>
-<wire x1="12.7" y1="154.94" x2="12.7" y2="157.48" width="0.1524" layer="91"/>
 <label x="12.7" y="157.48" size="1.778" layer="95" rot="R90" xref="yes"/>
 </segment>
@@
 <segment>
 <wire x1="50.8" y1="144.78" x2="50.8" y2="142.24" width="0.1524" layer="91"/>
-<wire x1="50.8" y1="142.24" x2="50.8" y2="137.16" width="0.1524" layer="91"/>
+<wire x1="50.8" y1="142.24" x2="50.8" y2="134.62" width="0.1524" layer="91"/>
 <wire x1="50.8" y1="142.24" x2="53.34" y2="142.24" width="0.1524" layer="91"/>
 <junction x="50.8" y="142.24"/>
@@
 </segment>
 <segment>
-<pinref part="GPSCONN" gate="G$1" pin="4"/>
 <wire x1="86.36" y1="88.9" x2="91.44" y2="88.9" width="0.1524" layer="91"/>
 <label x="91.44" y="88.9" size="1.778" layer="95"/>
+<pinref part="X5" gate="-4" pin="S"/>
 </segment>
 </net>
@@
 </segment>
 <segment>
-<pinref part="GPSCONN" gate="G$1" pin="3"/>
 <wire x1="86.36" y1="86.36" x2="91.44" y2="86.36" width="0.1524" layer="91"/>
 <label x="91.44" y="86.36" size="1.778" layer="95"/>
+<pinref part="X5" gate="-3" pin="S"/>
 </segment>
 </net>
@@
 <pinref part="C1" gate="G$1" pin="1"/>
 <pinref part="SUPPLY1" gate="G$1" pin="5V"/>
-<wire x1="33.02" y1="157.48" x2="33.02" y2="154.94" width="0.1524" layer="91"/>
 </segment>
 <segment>
@@
 </segment>
 <segment>
-<pinref part="GPSCONN" gate="G$1" pin="5"/>
 <wire x1="86.36" y1="91.44" x2="93.98" y2="91.44" width="0.1524" layer="91"/>
 <pinref part="SUPPLY5" gate="G$1" pin="5V"/>
 <wire x1="93.98" y1="91.44" x2="93.98" y2="96.52" width="0.1524" layer="91"/>
+<pinref part="X5" gate="-5" pin="S"/>
 </segment>
 </net>
@@
 </segment>
 <segment>
-<pinref part="GPSCONN" gate="G$1" pin="2"/>
 <wire x1="86.36" y1="83.82" x2="91.44" y2="83.82" width="0.1524" layer="91"/>
 <label x="91.44" y="83.82" size="1.778" layer="95"/>
+<pinref part="X5" gate="-2" pin="S"/>
 </segment>
 </net>
@@
 </segment>
 <segment>
-<pinref part="GPSCONN" gate="G$1" pin="1"/>
 <wire x1="86.36" y1="81.28" x2="91.44" y2="81.28" width="0.1524" layer="91"/>
 <label x="91.44" y="81.28" size="1.778" layer="95"/>
+<pinref part="X5" gate="-1" pin="S"/>
 </segment>
 </net>
@@
 </segment>
 <segment>
-<pinref part="U$2" gate="G$1" pin="3"/>
-<wire x1="20.32" y1="33.02" x2="12.7" y2="33.02" width="0.1524" layer="91"/>
-<label x="5.08" y="33.02" size="1.778" layer="95"/>
-</segment>
-</net>
+<pinref part="U$2" gate="G$1" pin="10"/>
+<wire x1="43.18" y1="17.78" x2="50.8" y2="17.78" width="0.1524" layer="91"/>
+<label x="50.8" y="17.78" size="1.778" layer="95"/>
+</segment>
+</net>
